File: RFPIGW.brd (EAGLE design)
At the start: 29.1 x 32.6 mm, 24 parts, among them U2 ATMEGA328

Commit message: Updated to V1.2
Parts:
- removed C4: 0.1uF, rcl:C0805
- removed PCS, PIRQ: (no value), jumper:SJ_2
- removed PVDD: (no value), jumper:SJ
- added U$2: RFM12B, _c2h:RFM12B-MINPADS
- added X1: 16MHz, SparkFun-FreqCtrl:RESONATOR-SMD
- C1: value 16MHz -> 0.1uF; device SparkFun-FreqCtrl:RESONATOR-SMD -> rcl:C0805
- OLED: device _c2h:1X04_LOCK -> _c2h:1X04_NO_LOCK
- U$4: value RFM69W -> AVR-ISP-6-EDGE; device _c2h:RFM69W-MINPADS -> avr-7:6PAD_ISP
- moved U$4 19.7 mm to (2.54, -2.54), flipped to the top, turned to 0 degrees
- moved ROOK69 11.7 mm to (11.6, 19.1)
- moved OLED 7.25 mm to (1.59, 17.8), turned to 270 degrees
- moved C1 6.15 mm to (5.46, 26.5), flipped to the top, turned to 90 degrees
- renumbered C5 to C3, C7 to C2
Connections:
- removed net +5V: ICSP.2, PVDD.1
- removed net CS12: PCS.2, U$3.SEL
- removed net IRQ12: PIRQ.2, U$3.IRQ
- net +3V3: now also C1.1, U$2.VDD; no longer C4.1, PVDD.2, U$4.VDD
- net D10: now also U$2.SEL; no longer PCS.3, U$4.NSS
- net D11/MOSI: now also U$2.SDI; no longer U$4.MISO
- net D12/MISO: now also U$2.SDO; no longer U$4.MOSI
- net D13/SCK: now also U$2.SCK; no longer U$4.SCK
- net D2: now also U$2.IRQ; no longer PIRQ.3, U$4.DIO0
- net D3: now also U$3.IRQ; no longer PIRQ.1
- net D5: now also U$3.SEL; no longer PCS.1
- net GND: now also U$2.GND, X1.2; no longer C4.2, U$4.GND
- net N$1: now also U$2.FSS; no longer U$4.DIO2
- net N$5: now also X1.1; no longer C1.1
- net N$6: now also U$2.ANT; no longer U$4.ANA
- net N$7: now also X1.3; no longer C1.3
Routing:
- net IRQ12: track 18.9 -> 0.00 mm, vias 1 -> 0
- net A0: track 25.9 -> 11.6 mm
- net A6: track 0.00 -> 14.0 mm, vias 0 -> 2
- net +3V3: track 91.6 -> 78.7 mm, vias 3 -> 2
- net CS12: track 12.8 -> 0.00 mm, vias 1 -> 0
- net D2: track 43.9 -> 31.6 mm, vias 3 -> 1
- net A7: track 0.00 -> 8.86 mm, vias 0 -> 2
- net D13/SCK: track 44.3 -> 52.5 mm
- net A4/SDA: track 29.4 -> 37.1 mm, vias 1 -> 2
- net D12/MISO: track 50.7 -> 43.1 mm
- net D5: track 12.9 -> 20.5 mm, vias 1 -> 0
- net RESET: track 61.3 -> 56.2 mm, vias 0 -> 1
- net D10: track 29.5 -> 24.6 mm
- net D3: track 13.9 -> 18.0 mm, vias 1 -> 2
- net N$1: track 13.1 -> 9.23 mm
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Other:
- board text added: "A6"
- board text added: "A7"
- board text added: "RFPIGW V1.2"
- board text added: "rssi"
- board text removed: "D2"
- board text removed: "D3"

Commit message: Updated to V1.2
Parts:
- removed ICSP: ISP 3V3, _c2h:2X3_LOCK
- removed ROOK12, ROOK69: 100, adafruit:R0805
- added ROOKBOT, ROOKTOP: 100, _c2h:0805-RES
- C1, C3: device rcl:C0805 -> _c2h:0805-CAP
- C2: device resistor:C0805 -> _c2h:0805-CAP
- LED1, LED2: value (none) -> LED0805-LARGE; device led:SML0805 -> _c2h:0805-LED-LARGEPADS
- R1, R2, R3: device adafruit:R0805 -> _c2h:0805-RES
- moved U$4 10.7 mm to (1.91, 8.13), turned to 90 degrees
- moved U$2 0.38 mm to (17.8, 8.00)
- moved R3 0.38 mm to (1.65, 27.2)
- moved LED2 0.13 mm to (2.41, 1.02)
- renumbered ANT to ANTTOP, ANT1 to ANTBOT
Connections:
- net +3V3: now also U$4.VCC
- net A0: now also ROOKBOT.1, ROOKTOP.1; no longer ROOK12.1, ROOK69.1
- net D11/MOSI: now also U$4.MOSI; no longer ICSP.4
- net D12/MISO: now also U$4.MISO; no longer ICSP.1
- net D13/SCK: now also U$4.SCK; no longer ICSP.3
- net D6: now also LED2.PLUS; no longer LED2.A
- net D9: now also LED1.PLUS; no longer LED1.A
- net GND: now also U$4.GND; no longer ICSP.6
- net N$1: now also ROOKBOT.2; no longer ROOK69.2
- net N$3: now also LED1.MINUS; no longer LED1.C
- net N$4: now also ROOKTOP.2; no longer ROOK12.2
- net N$8: now also LED2.MINUS; no longer LED2.C
- net RESET: now also U$4.RST; no longer ICSP.5
Routing:
- net +3V3: track 78.7 -> 106.4 mm, vias 2 -> 3
- net RESET: track 56.2 -> 43.7 mm, vias 1 -> 2
- net D12/MISO: track 43.1 -> 39.8 mm, vias 2 -> 3
- net D11/MOSI: track 44.4 -> 47.6 mm, vias 2 -> 3
- net N$1: track 9.23 -> 10.2 mm
- net N$8: track 6.63 -> 7.58 mm
- net D13/SCK: track 52.5 -> 51.9 mm
Other:
- board text added: "A1"
- board text added: "ANT"
- board text added: "D0"
- board text added: "D1"
- board text added: "D8"
- board text added: "MISO"
- board text added: "MOSI"
- board text added: "RFM69CW"
- board text added: "RST"
- board text added: "SCK"
- board text removed: "<"
- board text removed: "D10"
- board text removed: "D5"
- board text removed: "RFPIGW V1.1"
