File: RFPIGW.sch (EAGLE design)
At the start: 24 parts, among them U2 ATMEGA328

Commit message: Updated to V1.2
Parts:
- removed C4: 0.1uF, rcl:C-EUC0805
- removed PCS, PIRQ: (no value), jumper:SJ2W
- removed PVDD: (no value), jumper:SJ
- added U$2: RFM12B, _c2h:RFM12B
- added X1: 16MHz, SparkFun-FreqCtrl:RESONATOR16MHZ
- C1: value 16MHz -> 0.1uF; device SparkFun-FreqCtrl:RESONATOR16MHZ -> rcl:C-EUC0805
- U$4: value RFM69W -> AVR-ISP-6-EDGE; device _c2h:RFM69W -> avr-7:AVR-ISP-6-EDGE
- renumbered C5 to C3, C7 to C2
Connections:
- removed net +5V: ICSP.2, PVDD.1
- removed net CS12: PCS.2, U$3.SEL
- removed net IRQ12: PIRQ.2, U$3.IRQ
- net +3V3: now also C1.1, U$2.VCC; no longer C4.1, PVDD.2, U$4.VCC
- net D10: now also U$2.SEL; no longer PCS.3, U$4.SEL
- net D11/MOSI: now also U$2.SDI; no longer U$4.MISO
- net D12/MISO: now also U$2.SDO; no longer U$4.MOSI
- net D13/SCK: now also U$2.SCK; no longer U$4.SCK
- net D2: now also U$2.IRQ; no longer PIRQ.3, U$4.DIO0
- net D3: now also U$3.IRQ; no longer PIRQ.1
- net D5: now also U$3.SEL; no longer PCS.1
- net GND: now also U$2.GND, X1.2; no longer C4.2, U$4.GND
- net N$1: now also U$2.FFS; no longer U$4.DIO2
- net N$5: now also X1.1; no longer C1.1
- net N$6: now also U$2.ANT; no longer U$4.ANT
- net N$7: now also X1.3; no longer C1.3
Other:
- moved on the sheet: ANT1, ROOK69

Commit message: Updated to V1.2
Parts:
- removed ICSP: ISP 3V3, _c2h:AVR_SPI_PRG_62X3_LOCK
- removed ROOK12, ROOK69: 100, adafruit:R-US_R0805
- added ROOKBOT, ROOKTOP: 100, _c2h:RESISTOR0805-RES
- C1, C3: device rcl:C-EUC0805 -> _c2h:CAP0805-CAP
- C2: device resistor:C-EUC0805 -> _c2h:CAP0805-CAP
- LED1, LED2: value (none) -> LED0805-LARGE; device led:LEDSML0805 -> _c2h:LED0805-LARGE
- R1, R2, R3: device adafruit:R-US_R0805 -> _c2h:RESISTOR0805-RES
- renumbered ANT to ANTTOP, ANT1 to ANTBOT
Connections:
- net +3V3: now also U$4.P$6
- net A0: now also ROOKBOT.1, ROOKTOP.1; no longer ROOK12.1, ROOK69.1
- net D11/MOSI: now also U$4.P$5; no longer ICSP.4
- net D12/MISO: now also U$4.P$1; no longer ICSP.1
- net D13/SCK: now also U$4.P$2; no longer ICSP.3
- net D6: now also LED2.PLUS; no longer LED2.A
- net D9: now also LED1.PLUS; no longer LED1.A
- net GND: now also U$4.P$4; no longer ICSP.6
- net N$1: now also ROOKBOT.2; no longer ROOK69.2
- net N$3: now also LED1.MINUS; no longer LED1.C
- net N$4: now also ROOKTOP.2; no longer ROOK12.2
- net N$8: now also LED2.MINUS; no longer LED2.C
- net RESET: now also U$4.P$3; no longer ICSP.5
Other:
- note added: "RFM69CW"
- note added: "ROOKTOP and ROOKBOT only used for OOK mode of RFM12B/RFM69 OOK can be for RFM12B or RFM69 but not both at the same time"
- note added: "Take care if your ISP programmer power the board. Should be 3V3 Max if RF are on board if you don't want to burn them"
- note removed: "Close D10 and D2 if not using also a RFM69 device Close D5 and D3 if both RFM12B and RFM69 are present on the boardµ (and change pin definition in Arduino code)"
- note removed: "Close PVDD if you want your ISP programmer to power the board. Take care !!!!!! Should be 3V3 Max if RFM are on board if you don't want to burn RFM module"
- note removed: "ROOK12 and ROOK69 only used for OOK mode of RFM12B/RFM69 OOK can be for RFM12B or RFM69 but not both at the same time"
- moved on the sheet: C3
